Commit message: Versión definitiva 4 GDL: firmware fluido del usuario integrado + pick_place_node
El hardware definitivo es 4 GDL (yaw + 3 pitch) + gripper = 5 canales: el
antiguo roll fue retirado y su canal (servo GPIO 18 / pot GPIO 35) se
reutilizó para el pitch de muñeca.

- robotfun_firmware: firmware definitivo del usuario (tarea FreeRTOS de
  tiempo real a 50 Hz con perfil trapezoidal por junta y writeMicroseconds,
  pines SERVO {2,4,5,18,19} / POT {32,33,34,35,27}, RAW_ZERO
  {1267,1232,1265,1405,1302}, direcciones confirmadas). Único cambio: el
  canal 5 se publica como 'gripper' (antes 'joint_5') para coincidir con el
  URDF; /joint_command sigue siendo posicional [q1..q4, gripper].
- robotfun_kinematics: núcleo reestructurado a 4 GDL (A3=L3+L4=0.120,
  HAND=L5=0.090, FK(HOME)=[0.010,0,0.393], φ=π/2+q2+q3+q4); IK analítica
  cerrada + DLS/Newton/gradiente con reintentos; nuevo pick_place_node con
  la secuencia articular del usuario (waypoints probados a mano, duplicado
  de PLACE_OVER resuelto); nodos ik/trajectory/relay a 5 canales.
- robotfun_description: URDF de primitivas 4 GDL TF==FK (verificado contra
  el URDF real, error < 1e-12) y modelo de meshes del CAD; límites coherentes.
- README con comandos de clonado, verificación, simulación, pick & place y
  hardware; docs de arquitectura actualizadas.

Co-Authored-By: Claude Fable 5 <noreply@anthropic.com>
Claude-Session: https://claude.ai/code/session_01X9e4dopwyTqVmY9osf1kmo

File: src/robotfun_description/urdf/common/arm.macro.xacro (robot description, xacro)
@@ -1,20 +1,15 @@
 <?xml version="1.0"?>
 <!-- ============================================================================
-     arm.macro.xacro  —  esqueleto PRIMITIVO (tabla DH del usuario, 5 juntas)
+     arm.macro.xacro  —  esqueleto PRIMITIVO (tabla DH del usuario, 4 GDL)
      ===========================================================================
-     Brazo yaw + pitch + pitch + ROLL + pitch dibujado con PRIMITIVAS
-     dimensionadas a la tabla DH (metros):
-         L0=0.010  L1=0.063  L2=0.120  L3=0.090  L4=0.030  L5=0.090
+     Brazo 4 GDL RECTO (yaw + 3 pitch) dibujado con PRIMITIVAS dimensionadas a
+     la tabla DH (metros):
+         L0=0.010 (offset base)  L1=0.063  L2=0.120  A3=L3+L4=0.120  HAND=L5=0.090
      Reproduce EXACTAMENTE la FK del núcleo (TF == FK, validado por
      scripts/verify_kinematics.py y test_kinematics.py).
      FK(HOME) → TCP = [0.010, 0, 0.393].
-     Ejes (equivalencia URDF↔DH validada numéricamente):
-         joint_1 = (0 0 1)  yaw de base
-         joint_2 = (0 -1 0) pitch de hombro
-         joint_3 = (0 -1 0) pitch de codo
-         joint_4 = (0 0 1)  ROLL de muñeca (colineal con el antebrazo)
-         joint_5 = (0 +1 0) pitch de pinza  (signo + por la tabla DH: los dos
-                            twists α=+90° dejan el eje del pitch final en +Y)
+     Ejes: joint_1=(0 0 1) yaw; joint_2/3/4=(0 -1 0) pitch.
      tool0 = frame del TCP (punta del gripper), sin geometría.
+     La pinza apunta por el EJE X de tool0 (en HOME, hacia +Z).
      ========================================================================== -->
 <robot xmlns:xacro="http://www.ros.org/wiki/xacro">
@@ -71,39 +66,22 @@
       <axis xyz="0 -1 0"/><limit lower="${lo}" upper="${hi}" effort="10.0" velocity="1.5"/>
     </joint>
-    <!-- link_3: antebrazo inferior L3=0.090 (codo → servo de roll) -->
+    <!-- link_3: antebrazo A3=L3+L4=0.120 (codo → muñeca) -->
     <link name="link_3">
-      <inertial><origin xyz="0 0 0.045"/><mass value="0.2"/>
+      <inertial><origin xyz="0 0 0.06"/><mass value="0.3"/>
         <inertia ixx="8e-4" ixy="0" ixz="0" iyy="8e-4" iyz="0" izz="8e-4"/></inertial>
       <visual>
-        <origin xyz="0 0 0.045" rpy="0 0 0"/>
-        <geometry><cylinder radius="0.015" length="0.090"/></geometry>
+        <origin xyz="0 0 0.060" rpy="0 0 0"/>
+        <geometry><cylinder radius="0.015" length="0.120"/></geometry>
         <material name="blue"/>
       </visual>
     </link>
-    <!-- joint_4: ROLL de muñeca — eje colineal con el antebrazo (Z local).
-         En HOME girarlo NO traslada el TCP (roll puro, validado). -->
+    <!-- joint_4: pitch de muñeca/pinza -->
     <joint name="joint_4" type="revolute">
-      <origin xyz="0 0 0.090" rpy="0 0 0"/><parent link="link_3"/><child link="link_4"/>
-      <axis xyz="0 0 1"/><limit lower="${lo}" upper="${hi}" effort="10.0" velocity="1.5"/>
+      <origin xyz="0 0 0.120" rpy="0 0 0"/><parent link="link_3"/><child link="link_4"/>
+      <axis xyz="0 -1 0"/><limit lower="${lo}" upper="${hi}" effort="10.0" velocity="1.5"/>
     </joint>
-    <!-- link_4: antebrazo superior L4=0.030 (roll → pitch de pinza).
-         Caja (no cilindro) para VER girar el roll en RViz. -->
+    <!-- link_4: mano HAND=L5=0.090 (muñeca → punta del gripper) -->
     <link name="link_4">
-      <inertial><origin xyz="0 0 0.015"/><mass value="0.1"/>
-        <inertia ixx="5e-4" ixy="0" ixz="0" iyy="5e-4" iyz="0" izz="5e-4"/></inertial>
-      <visual>
-        <origin xyz="0 0 0.015" rpy="0 0 0"/>
-        <geometry><box size="0.030 0.018 0.030"/></geometry>
-        <material name="green"/>
-      </visual>
-    </link>
-    <!-- joint_5: pitch de pinza. Eje +Y (signo impuesto por la tabla DH). -->
-    <joint name="joint_5" type="revolute">
-      <origin xyz="0 0 0.030" rpy="0 0 0"/><parent link="link_4"/><child link="link_5"/>
-      <axis xyz="0 1 0"/><limit lower="${lo}" upper="${hi}" effort="10.0" velocity="1.5"/>
-    </joint>
-    <!-- link_5: mano L5=0.090 (pitch de pinza → punta del gripper) -->
-    <link name="link_5">
-      <inertial><origin xyz="0 0 0.045"/><mass value="0.15"/>
+      <inertial><origin xyz="0 0 0.045"/><mass value="0.2"/>
         <inertia ixx="5e-4" ixy="0" ixz="0" iyy="5e-4" iyz="0" izz="5e-4"/></inertial>
       <visual>
@@ -113,8 +91,7 @@
       </visual>
     </link>
-    <!-- tool0 = TCP (punta del gripper). Solo frame, sin geometría.
-         La pinza apunta por el EJE X de este frame (en HOME, hacia +Z). -->
+    <!-- tool0 = TCP (punta del gripper). Solo frame, sin geometría. -->
     <joint name="tool_fixed" type="fixed">
-      <origin xyz="0 0 0.090" rpy="0 0 0"/><parent link="link_5"/><child link="tool0"/>
+      <origin xyz="0 0 0.090" rpy="0 0 0"/><parent link="link_4"/><child link="tool0"/>
     </joint>
     <link name="tool0"/>

File: src/robotfun_description/urdf/robotfun.urdf.xacro (robot description, xacro)
@@ -3,7 +3,7 @@
      robotfun.urdf.xacro  —  MODELO DE MEDIDAS REALES (primitivas, tabla DH)
      ===========================================================================
-     Brazo de 5 juntas (yaw, pitch, pitch, ROLL, pitch) + gripper, con
-     PRIMITIVAS a las medidas de la tabla DH:
-         L0=0.010 L1=0.063 L2=0.120 L3=0.090 L4=0.030 L5=0.090  [m]
+     Brazo 4 GDL RECTO (yaw + 3 pitch) + gripper, con PRIMITIVAS a las medidas
+     de la tabla DH:
+         L0=0.010 L1=0.063 L2=0.120 A3=0.120 HAND=0.090  [m]
      Reproduce EXACTAMENTE la FK del núcleo (TF == FK): es el modelo canónico
      para VERIFICAR el DH y la cinemática inversa.
@@ -15,6 +15,6 @@
   <xacro:include filename="$(find robotfun_description)/urdf/common/gripper.macro.xacro"/>
   <xacro:robotfun_arm/>
-  <!-- gripper (canal 6) en la mano, cerca de la punta -->
-  <xacro:gripper_primitive parent="link_5">
+  <!-- gripper (canal 5 del firmware) en la mano, cerca de la punta -->
+  <xacro:gripper_primitive parent="link_4">
     <origin xyz="0 0 0.055" rpy="0 0 0"/>
   </xacro:gripper_primitive>

File: src/robotfun_description/urdf/robotfun_meshes.urdf.xacro (robot description, xacro)
@@ -6,16 +6,13 @@
      eslabon3 re-exportado y piezas unidas). Usa los orígenes de brazo.urdf
      (donde las mallas están alineadas) y la MISMA interfaz de juntas
-     (joint_1..joint_5 + gripper) y los MISMOS sentidos de giro que el modelo
-     primitivo, de modo que el mismo /joint_states mueve ambos modelos.
-     joint_4 (ROLL) se inserta en la muñeca con eje vertical en HOME (colineal
-     con el antebrazo): rota el conjunto muñeca+gripper (eslabon4) sobre sí
-     mismo. El eslabón portador link_4 no tiene visual (el CAD no tiene pieza
-     separada para el roll).
-     NOTA IMPORTANTE: las proporciones del CAD difieren de la tabla DH
-     (muñeca CAD a z=0.3865 vs 0.303 del DH; el offset x=0.038 del CAD es una
-     pieza descentrada del diseño original). El modelo PRIMITIVO
-     (model:=primitives) es la ÚNICA referencia válida para verificar
-     cinemática (TF == FK); este modelo es para VER el hardware. Si quieres
-     TF==FK también aquí, re-exporta las mallas a las longitudes L0..L5.
+     (joint_1..joint_4 + gripper implícito en eslabon4) que el modelo
+     primitivo, con los pitch en axis="0 -1 0" para el mismo sentido de giro.
+     Lo mueve el mismo /joint_states ⇒ la IK mueve también este modelo.
+     NOTA: las proporciones del CAD difieren de la tabla DH (muñeca CAD a
+     z=0.3865 vs 0.303 del DH; offset x=0.038 = pieza descentrada del diseño
+     original). El modelo PRIMITIVO (model:=primitives) es la ÚNICA referencia
+     válida para verificar cinemática (TF == FK); este modelo es para VER el
+     hardware. El gripper real es parte de eslabon4 (piezas unidas): no tiene
+     junta 'gripper' propia en este modelo.
      ========================================================================== -->
 <robot name="robotfun_meshes" xmlns:xacro="http://www.ros.org/wiki/xacro">
@@ -70,20 +67,10 @@
     </visual>
   </link>
-  <!-- joint_4: ROLL de muñeca (nuevo respecto a brazo.urdf). El eje pasa por
-       el centro de la muñeca del CAD (x=0.038 en el frame de link_3: pieza
-       descentrada del diseño original) y es vertical en HOME. -->
   <joint name="joint_4" type="revolute">
     <origin xyz="0.038 0 0.1213" rpy="0 0 0"/><parent link="link_3"/><child link="link_4"/>
-    <axis xyz="0 0 1"/><limit lower="${lo}" upper="${hi}" effort="10.0" velocity="1.5"/>
+    <axis xyz="0 -1 0"/><limit lower="${lo}" upper="${hi}" effort="10.0" velocity="1.5"/>
   </joint>
-  <!-- link_4: portador del roll (el CAD no tiene pieza separada) -->
-  <link name="link_4"/>
-  <!-- joint_5: pitch de pinza. Eje +Y, igual que el modelo primitivo/DH. -->
-  <joint name="joint_5" type="revolute">
-    <origin xyz="0 0 0" rpy="0 0 0"/><parent link="link_4"/><child link="link_5"/>
-    <axis xyz="0 1 0"/><limit lower="${lo}" upper="${hi}" effort="10.0" velocity="1.5"/>
-  </joint>
-  <!-- link_5 = eslabon4 del CAD (muñeca + gripper unidos en una pieza) -->
-  <link name="link_5">
+  <!-- link_4 = eslabon4 (muñeca + gripper unidos: un solo eslabón) -->
+  <link name="link_4">
     <visual>
       <origin xyz="-0.038 0 -0.3865" rpy="0 0 0"/>
@@ -92,7 +79,7 @@
     </visual>
   </link>
-  <!-- tool0 = TCP (punta del gripper, L5=0.090). Solo frame. -->
+  <!-- tool0 = TCP (punta del gripper, HAND=L5=0.090). Solo frame. -->
   <joint name="tool_fixed" type="fixed">
-    <origin xyz="0 0 0.090" rpy="0 0 0"/><parent link="link_5"/><child link="tool0"/>
+    <origin xyz="0 0 0.090" rpy="0 0 0"/><parent link="link_4"/><child link="tool0"/>
   </joint>
   <link name="tool0"/>
